Commit message: update joint limits

File: urdf/scope89_ptz.urdf (robot description, URDF)
Before this commit: robot scope89_ptz, 3 links, 2 joints
Joints:
- joint J1: limit lower=0 upper=0 effort=0 velocity=0 -> lower=-3.1415 upper=3.1415 effort=10 velocity=1.0
- joint J2: limit lower=0 upper=0 effort=0 velocity=0 -> lower=-2.443 upper=2.443 effort=10 velocity=1.0
